File: anubis.sch (KiCad schematic (older format))
At the start: 12 parts, among them J1 Conn_02x20_Odd_Even

Commit message: make it good
Parts:
- added C1, C2, C3, C4: 0.1uF, Capacitor_SMD:C_0805_2012Metric_Pad1.15x1.40mm_HandSolder, symbol Device:C
- added R1, R2: 10K, Resistor_SMD:R_0805_2012Metric_Pad1.15x1.40mm_HandSolder, symbol Device:R
- added unit 2 of U9
- added unit 7 of U9
- added unit 3 of U9
- added unit 4 of U9
- added unit 5 of U9
- added unit 6 of U9
- J1: footprint (none) -> Connector_PinSocket_2.54mm:PinSocket_2x20_P2.54mm_Vertical
- J2: renamed from J?; footprint (none) -> Connector_PinSocket_2.54mm:PinSocket_2x20_P2.54mm_Vertical
- U1, U2, U3, U4, U5, U6, U7, U8: renamed from U?; footprint SOIC127P1030X265-24N -> Package_SO:SOIC-24W_7.5x15.4mm_P1.27mm
- U10: renamed from U?; footprint (none) -> anubis:DIP-64_750_ELL
- U9: renamed from U?; footprint (none) -> Package_SO:SOIC-14_3.9x8.7mm_P1.27mm
Connections:
- wire segments 36 -> 54
- no-connect marks 0 -> 1
Other:
- moved on the sheet: J2

Commit message: fix some part numbers
Parts:
- U9: value 74LS05 -> 74LV05
Other:
- note added: "Flipped left-to-right!"
Changed lines of the file:
@@
 EESchema Schematic File Version 4
-LIBS:anubis-cache
-EELAYER 29 0
+EELAYER 30 0
 EELAYER END
 $Descr B 17000 11000
@@
 P 10650 6550
 F 0 "U9" H 10650 6867 50  0000 C CNN
-F 1 "74LS05" H 10650 6776 50  0000 C CNN
+F 1 "74LV05" H 10650 6776 50  0000 C CNN
 F 2 "Package_SO:SOIC-14_3.9x8.7mm_P1.27mm" H 10650 6550 50  0001 C CNN
 F 3 "http://www.ti.com/lit/gpn/sn74LS05" H 10650 6550 50  0001 C CNN
@@
 P 10600 5800
 F 0 "U9" H 10600 6117 50  0000 C CNN
-F 1 "74LS05" H 10600 6026 50  0000 C CNN
+F 1 "74LV05" H 10600 6026 50  0000 C CNN
 F 2 "Package_SO:SOIC-14_3.9x8.7mm_P1.27mm" H 10600 5800 50  0001 C CNN
 F 3 "http://www.ti.com/lit/gpn/sn74LS05" H 10600 5800 50  0001 C CNN
@@
 P 10600 4700
 F 0 "U9" H 10830 4746 50  0000 L CNN
-F 1 "74LS05" H 10830 4655 50  0000 L CNN
+F 1 "74LV05" H 10830 4655 50  0000 L CNN
 F 2 "Package_SO:SOIC-14_3.9x8.7mm_P1.27mm" H 10600 4700 50  0001 C CNN
 F 3 "http://www.ti.com/lit/gpn/sn74LS05" H 10600 4700 50  0001 C CNN
@@
 P 10650 7850
 F 0 "U9" H 10650 8167 50  0000 C CNN
-F 1 "74LS05" H 10650 8076 50  0000 C CNN
+F 1 "74LV05" H 10650 8076 50  0000 C CNN
 F 2 "Package_SO:SOIC-14_3.9x8.7mm_P1.27mm" H 10650 7850 50  0001 C CNN
 F 3 "http://www.ti.com/lit/gpn/sn74LS05" H 10650 7850 50  0001 C CNN
@@
 P 10650 8400
 F 0 "U9" H 10650 8717 50  0000 C CNN
-F 1 "74LS05" H 10650 8626 50  0000 C CNN
+F 1 "74LV05" H 10650 8626 50  0000 C CNN
 F 2 "Package_SO:SOIC-14_3.9x8.7mm_P1.27mm" H 10650 8400 50  0001 C CNN
 F 3 "http://www.ti.com/lit/gpn/sn74LS05" H 10650 8400 50  0001 C CNN
@@
 P 10650 8950
 F 0 "U9" H 10650 9267 50  0000 C CNN
-F 1 "74LS05" H 10650 9176 50  0000 C CNN
+F 1 "74LV05" H 10650 9176 50  0000 C CNN
 F 2 "Package_SO:SOIC-14_3.9x8.7mm_P1.27mm" H 10650 8950 50  0001 C CNN
 F 3 "http://www.ti.com/lit/gpn/sn74LS05" H 10650 8950 50  0001 C CNN
@@
 P 10650 9500
 F 0 "U9" H 10650 9817 50  0000 C CNN
-F 1 "74LS05" H 10650 9726 50  0000 C CNN
+F 1 "74LV05" H 10650 9726 50  0000 C CNN
 F 2 "Package_SO:SOIC-14_3.9x8.7mm_P1.27mm" H 10650 9500 50  0001 C CNN
 F 3 "http://www.ti.com/lit/gpn/sn74LS05" H 10650 9500 50  0001 C CNN
@@
 Wire Wire Line
 	15300 7500 15500 7500
+Text Notes 1050 2550 0    50   ~ 0
+Flipped left-to-right!
 $EndSCHEMATC
